Commit message: working urdf model of mechanum car

File: urdf/mechanum_car.xacro.urdf (robot description, URDF)
Before this commit: robot mechanum_car, 2 links, 1 joints
Links:
- added link back_left_wheel, mass 100; collision cylinder length=0.05 radius=0.07; visual cylinder length=0.05 radius=0.07
- added link back_right_wheel, mass 100; collision cylinder length=0.05 radius=0.07; visual cylinder length=0.05 radius=0.07
- added link front_right_wheel, mass 100; collision cylinder length=0.05 radius=0.07; visual cylinder length=0.05 radius=0.07
- added link world
- link front_left_wheel: mass None -> 100
- link mechanum_chasis: mass None -> 100
Joints:
- added joint back_left_hinge: type continuous, parent mechanum_chasis, child back_left_wheel, origin xyz=0.1 -0.1 -0.03 rpy=0 -1.5708 0, axis 0.0 0.0 1.0
- added joint back_right_hinge: type continuous, parent mechanum_chasis, child back_right_wheel, origin xyz=-0.1 -0.1 -0.03 rpy=0 -1.5708 0, axis 0.0 0.0 1.0
- added joint front_right_hinge: type continuous, parent mechanum_chasis, child front_right_wheel, origin xyz=-0.1 0.1 -0.03 rpy=0 -1.5708 0, axis 0.0 0.0 1.0
- added joint world_to_base: type fixed, parent world, child mechanum_chasis, origin xyz=0 0 0.1 rpy=0 0 0
