Commit message: Fix problem where robot can't move
The robot was not able to move cause of the fixed joint to the world
frame, but can use the pose tag of a link to make sure the model doesn't
fall through the world, adding some xacro properties, still need to
figure out how to make gazebo_ros use the parse version of the urdf xml.

File: urdf/mecanum_car.xacro.urdf (robot description, URDF)
Before this commit: robot mechanum_car, 6 links, 5 joints
Links:
- removed link mechanum_chasis
- removed link world
- added link mecanum_chasis, mass 1; collision box size=0.15 0.35 0.08; visual box size=${chasis_width} ${chasis_length} ${chasis_height}
- link back_left_wheel: mass 100 -> 1
- link back_right_wheel: mass 100 -> 1
- link front_left_wheel: mass 100 -> 1
- link front_right_wheel: mass 100 -> 1
Joints:
- removed joint world_to_base
- joint back_left_hinge: parent mechanum_chasis -> mecanum_chasis
- joint back_right_hinge: parent mechanum_chasis -> mecanum_chasis
- joint front_left_hinge: parent mechanum_chasis -> mecanum_chasis
- joint front_right_hinge: parent mechanum_chasis -> mecanum_chasis

Commit message: simplified model urdf with xacro macros

File: urdf/mecanum_car.xacro.urdf (robot description, URDF)
Before this commit: robot mecanum_car, 5 links, 4 joints
Links:
- removed link back_left_wheel
- removed link back_right_wheel
- removed link front_left_wheel
- removed link front_right_wheel
Joints:
- removed joint back_left_hinge
- removed joint back_right_hinge
- removed joint front_left_hinge
- removed joint front_right_hinge

Commit message: working joystick control

File: urdf/mecanum_car.xacro.urdf (robot description, URDF)
Before this commit: robot mecanum_car, 1 links, 0 joints
Links:
- added link base_footprint
Joints:
- added joint base_joint: type fixed, parent base_footprint, child mecanum_chasis, origin xyz=0.0 0.0 ${-(wheel_radius+wheel_zoff)} rpy=0 0 0

Commit message: workng visual meshes

File: urdf/mecanum_car.xacro.urdf (robot description, URDF)
Before this commit: robot mecanum_car, 2 links, 1 joints
Joints:
- joint base_joint: origin xyz=0.0 0.0 ${-(wheel_radius+wheel_zoff)} rpy=0 0 0 -> xyz=0.0 0.0 ${-(0.07+wheel_zoff)} rpy=0 0 0

Commit message: simplified model urdf to not use wheel mesh

File: urdf/mecanum_car.xacro.urdf (robot description, URDF)
Before this commit: robot mecanum_car, 2 links, 1 joints
Links:
- removed link mecanum_chasis
- added link base_link, mass 1; collision box size=${chasis_width} ${chasis_length} ${chasis_height}; visual box size=${chasis_width} ${chasis_length} ${chasis_height}
Joints:
- joint base_joint: child mecanum_chasis -> base_footprint; parent base_footprint -> base_link

Commit message: added gazebo launch and imu sensors

File: urdf/mecanum_car.xacro.urdf (robot description, URDF)
Before this commit: robot mecanum_car, 2 links, 1 joints
Links:
- added link imu_link; collision box size=0.025 0.025 0.025; visual box size=0.025 0.025 0.025
Joints:
- added joint imu_joint: type fixed, parent base_link, child imu_link, origin xyz=0 0 0.05
