Commit message: Function launch of gazebo
Launching gazebo with launch files with specified world and model

File: urdf/diff_drive.xacro.urdf (robot description, URDF)
Before this commit: robot diff_drive, 7 links, 6 joints
Links:
- removed link camera_depth_frame
- removed link camera_link
- removed link imu_link
- removed link lidar_link
Joints:
- removed joint camera_depth_joint
- removed joint camera_joint
- removed joint imu_joint
- removed joint lidar_joint
